Commit message: Fix hardware_interface / description

File: arctos_hardware_interface/ros2_control/arctos.ros2_control.xacro (robot description, xacro)
@@ -6,5 +6,5 @@
         <plugin>libarctos_interface.so</plugin>
       </hardware>
-      <joint name="joint_1">
+      <joint name="X_joint">
         <command_interface name="position">
           <param name="min">{-2*pi}</param>
@@ -20,5 +20,5 @@
         <state_interface name="velocity"/>
       </joint>
-      <joint name="joint_2">
+      <joint name="Y_joint">
         <command_interface name="position">
           <param name="min">{-2*pi}</param>
@@ -34,5 +34,5 @@
         <state_interface name="velocity"/>
       </joint>
-      <joint name="joint_3">
+      <joint name="Z_joint">
         <command_interface name="position">
           <param name="min">{-pi}</param>
@@ -48,5 +48,5 @@
         <state_interface name="velocity"/>
       </joint>
-      <joint name="joint_4">
+      <joint name="A_joint">
         <command_interface name="position">
           <param name="min">{-2*pi}</param>
@@ -62,5 +62,5 @@
         <state_interface name="velocity"/>
       </joint>
-      <joint name="joint_5">
+      <joint name="B_joint">
         <command_interface name="position">
           <param name="min">{-2*pi}</param>
@@ -76,5 +76,5 @@
         <state_interface name="velocity"/>
       </joint>
-      <joint name="joint_6">
+      <joint name="C_joint">
         <command_interface name="position">
           <param name="min">{-2*pi}</param>
