Commit message: Joint states are now being properly updated in the motor driver. The states will be updated only after the motors have performed the requested action. (e.g. move to a position, home, etc.)
There is currently a bug in the motor driver due to the backlash of the gearbox.
The position of N joint can unexpectedly change to a value when no command is issued, likely due to gearbox backlash​.
This is a known issue and will be addressed in the future.

- Add `hardware_type` to the motor config file (MKS_42D, MKS_57D)
    - This is to be able to know when the endstop limit switches are triggered.
- Add `gear_ratio` to the motor config file

File: arctos_description/urdf/test_single_motor.urdf.xacro (robot description, xacro)
@@ -19,4 +19,9 @@
       <state_interface name="velocity"/>
     </joint>
+    <joint name="joint_y">
+      <command_interface name="position"/>
+      <state_interface name="position"/>
+      <state_interface name="velocity"/>
+    </joint>
   </ros2_control>
 </robot>
