Commit message: Update urdf issues

File: arctos_description/urdf/arctos.xacro (robot description, xacro)
@@ -3,5 +3,5 @@
   <xacro:include filename="$(find arctos_description)/urdf/materials.xacro" />
   <xacro:include filename="$(find arctos_description)/urdf/joint_link.xacro" />
-  <xacro:include filename="$(find arctos_description)/urdf/arctos.ros2_control.xacro" />
+  <xacro:include filename="$(find arctos_description)/urdf/arctos_ros2_control.xacro" />
   <xacro:include filename="$(find arctos_description)/urdf/arctos_gripper.xacro" />
   <!-- Define all links -->

File: arctos_description/urdf/arctos_gripper.xacro (robot description, xacro)
@@ -27,31 +27,26 @@
     ixx="0.0" iyy="0.0" izz="0.0" ixy="-0.0" iyz="0.0" ixz="0.0"
   />
+  <!-- Fixed gripper joint, no axis needed -->
   <xacro:arctos_joint
     name="Gripper_joint" type="fixed"
     parent="Link_6_1" child="Gripper_1"
     origin_xyz="0.0 -0.0 0.0" origin_rpy="0 0 0"
-    axis_xyz="1.0 0.0 -0.0"
     limit_u="0.0" limit_l="0.0" limit_e="0.0" limit_v="0.0"
   />
-  <xacro:arctos_joint
-    name="Left_jaw_joint" type="prismatic"
-    parent="Gripper_1" child="Left_jaw_1"
-    origin_xyz="0.0 -0.0 0.0" origin_rpy="0 0 0"
-    axis_xyz="0.0 0.0 -1.0"
-    limit_u="0.015" limit_l="0.0" limit_e="1.0" limit_v="10.0"
-  />
+  <!-- Left jaw joint, prismatic with axis directly defined -->
+  <joint name="Left_jaw_joint" type="prismatic">
+    <parent link="Gripper_1"/>
+    <child link="Left_jaw_1"/>
+    <origin xyz="0.0 0.0 0.0" rpy="0 0 0"/>
+    <axis xyz="0.0 0.0 -1.0"/>
+    <limit effort="1.0" lower="0.0" upper="0.015" velocity="10.0"/>
+  </joint>
+  <!-- Right jaw joint, prismatic with axis directly defined -->
   <joint name="Right_jaw_joint" type="prismatic">
-    <mimic joint="Left_jaw_joint" multiplier="-1.0" offset="0" />
-    <axis xyz="0 0 -1" />
-    <origin xyz="0.0 0.0 0." rpy="0.0 0.0 0.0" />
-    <parent link="Gripper_1" />
-    <child link="Right_jaw_1" />
-    <limit effort="1.0" lower="0" upper="0.1" velocity="10.0" />
+    <parent link="Gripper_1"/>
+    <child link="Right_jaw_1"/>
+    <origin xyz="0.0 0.0 0.0" rpy="0 0 0"/>
+    <axis xyz="0.0 0.0 -1.0"/>
+    <limit effort="1.0" lower="0.0" upper="0.1" velocity="10.0"/>
   </joint>
-  <xacro:arctos_control
-    name="Left_jaw_joint"
-    can_id="0x07"
-    limit_u="0.015"
-    limit_l="0.0"
-  />
 </robot>

File: arctos_description/urdf/arctos_ros2_control.xacro (robot description, xacro)
@@ -4,5 +4,5 @@
     <ros2_control name="${name}" type="system">
       <hardware>
-        <plugin>libarctos_interface.so</plugin>
+        <plugin>arctos_interface/ArctosInterface</plugin>
       </hardware>
       <joint name="X_joint">

File: arctos_description/urdf/joint_link.xacro (robot description, xacro)
@@ -34,102 +34,3 @@
     </joint>
   </xacro:macro>
-  <xacro:macro name="arctos_control" params="name can_id limit_u limit_l">
-  <ros2_control name="arctos" type="system">
-    <hardware>
-      <plugin>arctos_interface/ArctosInterface</plugin>
-    </hardware>
-    <joint name="X_joint">
-      <command_interface name="position">
-        <param name="min">{-2*pi}</param>
-        <param name="max">{2*pi}</param>
-      </command_interface>
-      <command_interface name="velocity">
-        <param name="min">-3.15</param>
-        <param name="max">3.15</param>
-      </command_interface>
-      <state_interface name="position">
-        <param name="initial_value">0.0</param>
-      </state_interface>
-      <state_interface name="velocity"/>
-    </joint>
-    <joint name="Y_joint">
-      <command_interface name="position">
-        <param name="min">{-2*pi}</param>
-        <param name="max">{2*pi}</param>
-      </command_interface>
-      <command_interface name="velocity">
-        <param name="min">-3.15</param>
-        <param name="max">3.15</param>
-      </command_interface>
-      <state_interface name="position">
-        <param name="initial_value">0.0</param>
-      </state_interface>
-      <state_interface name="velocity"/>
-    </joint>
-    <joint name="Z_joint">
-      <command_interface name="position">
-        <param name="min">{-pi}</param>
-        <param name="max">{pi}</param>
-      </command_interface>
-      <command_interface name="velocity">
-        <param name="min">-3.15</param>
-        <param name="max">3.15</param>
-      </command_interface>
-      <state_interface name="position">
-        <param name="initial_value">0.0</param>
-      </state_interface>
-      <state_interface name="velocity"/>
-    </joint>
-    <joint name="A_joint">
-      <command_interface name="position">
-        <param name="min">{-2*pi}</param>
-        <param name="max">{2*pi}</param>
-      </command_interface>
-      <command_interface name="velocity">
-        <param name="min">-3.2</param>
-        <param name="max">3.2</param>
-      </command_interface>
-      <state_interface name="position">
-        <param name="initial_value">0.0</param>
-      </state_interface>
-      <state_interface name="velocity"/>
-    </joint>
-    <joint name="B_joint">
-      <command_interface name="position">
-        <param name="min">{-2*pi}</param>
-        <param name="max">{2*pi}</param>
-      </command_interface>
-      <command_interface name="velocity">
-        <param name="min">-3.2</param>
-        <param name="max">3.2</param>
-      </command_interface>
-      <state_interface name="position">
-        <param name="initial_value">0.0</param>
-      </state_interface>
-      <state_interface name="velocity"/>
-    </joint>
-    <joint name="C_joint">
-      <command_interface name="position">
-        <param name="min">{-2*pi}</param>
-        <param name="max">{2*pi}</param>
-      </command_interface>
-      <command_interface name="velocity">
-        <param name="min">-3.2</param>
-        <param name="max">3.2</param>
-      </command_interface>
-      <state_interface name="position">
-        <param name="initial_value">0.0</param>
-      </state_interface>
-      <state_interface name="velocity"/>
-    </joint>
-    <sensor name="tcp_fts_sensor">
-      <state_interface name="force.x"/>
-      <state_interface name="force.y"/>
-      <state_interface name="force.z"/>
-      <state_interface name="torque.x"/>
-      <state_interface name="torque.y"/>
-      <state_interface name="torque.z"/>
-    </sensor>
-  </ros2_control>
-  </xacro:macro>
 </robot>

File: arctos_hardware_interface/ros2_control/arctos.ros2_control.xacro (robot description, xacro)
@@ -16,5 +16,5 @@
         </command_interface>
         <state_interface name="position">
-          <param name="initial_value">0.0</param>arctos.ros2_control.xacro
+          <param name="initial_value">0.0</param>
         </state_interface>
         <state_interface name="velocity"/>

Commit message: Trying plugin corrections

File: arctos_description/urdf/arctos.xacro (robot description, xacro)
@@ -117,3 +117,4 @@
     limit_u="${pi}" limit_l="${-pi}" limit_e="16.0" limit_v="3.0"
   />
+  <xacro:arctos_ros2_control name="arctos_interface" />
 </robot>

File: arctos_description/urdf/arctos_gripper.xacro (robot description, xacro)
@@ -35,18 +35,29 @@
   />
   <!-- Left jaw joint, prismatic with axis directly defined -->
-  <joint name="Left_jaw_joint" type="prismatic">
-    <parent link="Gripper_1"/>
-    <child link="Left_jaw_1"/>
-    <origin xyz="0.0 0.0 0.0" rpy="0 0 0"/>
-    <axis xyz="0.0 0.0 -1.0"/>
-    <limit effort="1.0" lower="0.0" upper="0.015" velocity="10.0"/>
-  </joint>
-  <!-- Right jaw joint, prismatic with axis directly defined -->
-  <joint name="Right_jaw_joint" type="prismatic">
-    <parent link="Gripper_1"/>
-    <child link="Right_jaw_1"/>
-    <origin xyz="0.0 0.0 0.0" rpy="0 0 0"/>
-    <axis xyz="0.0 0.0 -1.0"/>
-    <limit effort="1.0" lower="0.0" upper="0.1" velocity="10.0"/>
-  </joint>
+  <xacro:arctos_joint
+    name="Left_jaw_joint"
+    type="prismatic"
+    parent="Gripper_1"
+    child="Left_jaw_1"
+    origin_xyz="0.0 0.0 0.0"
+    origin_rpy="0 0 0"
+    axis_xyz="0 0 1"
+    limit_u="0.015"
+    limit_l="0.0"
+    limit_e="1.0"
+    limit_v="10.0"
+  />
+  <xacro:arctos_joint
+    name="Right_jaw_joint"
+    type="prismatic"
+    parent="Gripper_1"
+    child="Right_jaw_1"
+    origin_xyz="0.0 0.0 0.0"
+    origin_rpy="0 0 0"
+    axis_xyz="0 0 1"
+    limit_u="0.015"
+    limit_l="0.0"
+    limit_e="1.0"
+    limit_v="10.0"
+  />
 </robot>

File: arctos_description/urdf/joint_link.xacro (robot description, xacro)
@@ -1,4 +1,5 @@
 <?xml version="1.0"?>
 <robot xmlns:xacro="http://www.ros.org/wiki/xacro" name="arctos">
+  <!-- Define arctos_link macro -->
   <xacro:macro name="arctos_link"
     params="name origin_xyz origin_rpy material_name inertia_origin_xyz inertia_origin_rpy mass ixx iyy izz ixy iyz ixz">
@@ -24,6 +25,7 @@
     </link>
   </xacro:macro>
+  <!-- Define arctos_joint macro with a default value for axis_xyz -->
   <xacro:macro name="arctos_joint"
-    params="name type parent child origin_xyz origin_rpy axis_xyz limit_u limit_l limit_e limit_v">
+    params="name type parent child origin_xyz origin_rpy axis_xyz='0 0 0' limit_u limit_l limit_e limit_v">
     <joint name="${name}" type="${type}">
       <parent link="${parent}" />

File: arctos_hardware_interface/ros2_control/arctos.ros2_control.xacro (robot description, xacro)
@@ -4,5 +4,5 @@
     <ros2_control name="${name}" type="system">
       <hardware>
-        <plugin>libarctos_interface.so</plugin>
+        <plugin>lib/libarctos_interface</plugin>
       </hardware>
       <joint name="X_joint">

Commit message: Still need to work on:
- Ensure set_zero_position.py returns Z to the home opposition to prevent the arm from crashing.
- Make a function dedicated to the movement of B/C.
- Test RVIZ/move it with the new changes (Since my robot doesn't have A, B, C right now, I had to focus on re-assembling it).

File: arctos_description/urdf/arctos.xacro (robot description, xacro)
@@ -100,5 +100,5 @@
     parent="Link_3_1" child="Link_4_1"
     origin_xyz="0 -0.13881 0.0217651" origin_rpy="0 0 0"
-    axis_xyz="-0.0 1.0 -0.0"
+    axis_xyz="0.0 1.0 0.0"
     limit_u="${pi}" limit_l="${-pi}" limit_e="22.0" limit_v="4.4"
   />
@@ -107,5 +107,5 @@
     parent="Link_4_1" child="Link_5_1"
     origin_xyz="0.0 -0.12543 -0.00184" origin_rpy="0 0 0"
-    axis_xyz="-1.0 -0.0 0.0"
+    axis_xyz="-1.0 0.0 0.0"
     limit_u="1.55" limit_l="-1.55" limit_e="16.0" limit_v="3.0"
   />
@@ -114,5 +114,5 @@
     parent="Link_5_1" child="Link_6_1"
     origin_xyz="0.0 -0.0398 0.0" origin_rpy="0 0 0"
-    axis_xyz="-0.0 1.0 -0.0"
+    axis_xyz="0.0 1.0 0.0"
     limit_u="${pi}" limit_l="${-pi}" limit_e="16.0" limit_v="3.0"
   />

File: arctos_description/urdf/arctos_ros2_control.xacro (robot description, xacro)
@@ -2,50 +2,21 @@
 <robot xmlns:xacro="http://www.ros.org/wiki/xacro">
   <xacro:macro name="arctos_ros2_control" params="name">
+    <xacro:include filename="$(find arctos_description)/urdf/joint_link.xacro"/>
     <ros2_control name="${name}" type="system">
       <hardware>
         <plugin>arctos_interface/ArctosInterface</plugin>
       </hardware>
-      <joint name="X_joint">
-        <command_interface name="position">
-          <param name="min">{-2*pi}</param>
-          <param name="max">{2*pi}</param>
-        </command_interface>
-        <command_interface name="velocity">
-          <param name="min">-3.15</param>
-          <param name="max">3.15</param>
-        </command_interface>
-        <state_interface name="position">
-          <param name="initial_value">0.0</param>
-        </state_interface>
-        <state_interface name="velocity"/>
-      </joint>
-      <joint name="Y_joint">
-        <command_interface name="position">
-          <param name="min">{-2*pi}</param>
-          <param name="max">{2*pi}</param>
-        </command_interface>
-        <command_interface name="velocity">
-          <param name="min">-3.15</param>
-          <param name="max">3.15</param>
-        </command_interface>
-        <state_interface name="position">
-          <param name="initial_value">0.0</param>
-        </state_interface>
-        <state_interface name="velocity"/>
-      </joint>
-      <joint name="Z_joint">
-        <command_interface name="position">
-          <param name="min">{-pi}</param>
-          <param name="max">{pi}</param>
-        </command_interface>
-        <command_interface name="velocity">
-          <param name="min">-3.15</param>
-          <param name="max">3.15</param>
-        </command_interface>
-        <state_interface name="position">
-          <param name="initial_value">0.0</param>
-        </state_interface>
-        <state_interface name="velocity"/>
-      </joint>
+      <xacro:arctos_control
+        name="X_joint"
+        limit_u="${pi}" limit_l="${-pi}"
+      />
+      <xacro:arctos_control
+        name="Y_joint"
+        limit_u="-0.88" limit_l="1.97"
+      />
+      <xacro:arctos_control
+        name="Z_joint"
+        limit_u="0.65" limit_l="-1.6"
+      />
       <joint name="A_joint">
         <command_interface name="position">

File: arctos_description/urdf/joint_link.xacro (robot description, xacro)
@@ -35,4 +35,24 @@
       <limit upper="${limit_u}" lower="${limit_l}" effort="${limit_e}" velocity="${limit_v}" />
     </joint>
+    <!-- Add transmission element -->
+    <transmission name="transmission_${name}">
+      <type>transmission_interface/SimpleTransmission</type>
+      <joint name="${name}">
+        <hardwareInterface>hardware_interface/PositionJointInterface</hardwareInterface>
+      </joint>
+      <actuator name="${name}_motor">
+        <mechanicalReduction>1.0</mechanicalReduction>
+      </actuator>
+    </transmission>
+  </xacro:macro>
+  <xacro:macro name="arctos_control" params="name limit_u limit_l">
+    <joint name="${name}">
+      <command_interface name="position">
+            <param name="min">${limit_l}</param>
+            <param name="max">${limit_u}</param>
+      </command_interface>
+      <state_interface name="position"/>
+      <state_interface name="velocity"/>
+    </joint>
   </xacro:macro>
 </robot>

Commit message: Use 6 joints configuration

File: arctos_description/urdf/arctos.xacro (robot description, xacro)
@@ -72,4 +72,5 @@
     ixx="1e-3" iyy="1e-3" izz="1e-3" ixy="-0.0" iyz="0.0" ixz="0.0"
   />
+  <!--Change limit of joints here-->
   <xacro:arctos_joint
     name="X_joint" type="revolute"
@@ -91,5 +92,5 @@
     origin_xyz="0.0 0.001365 0.261035" origin_rpy="0 0 0"
     axis_xyz="1.0 -0.0 0.0"
-    limit_u="${70/180*pi}" limit_l="${-pi/2}" limit_e="97.0" limit_v="1.4"
+    limit_u="${55/180*pi}" limit_l="${-pi/2}" limit_e="97.0" limit_v="1.4"
   />
   <xacro:arctos_joint
@@ -98,5 +99,5 @@
     origin_xyz="0 -0.13881 0.0217651" origin_rpy="0 0 0"
     axis_xyz="0.0 1.0 0.0"
-    limit_u="${pi}" limit_l="${-pi}" limit_e="22.0" limit_v="4.4"
+    limit_u="${pi/2}" limit_l="${-pi/2}" limit_e="22.0" limit_v="4.4"
   />
   <xacro:arctos_joint

File: arctos_description/urdf/arctos_gripper.xacro (robot description, xacro)
@@ -6,25 +6,25 @@
   <xacro:arctos_link
     name="Gripper_1"
-    origin_xyz="0.0 0.323 -0.5685" origin_rpy="0 0 0"
+    origin_xyz="-0.000193 0.319847 -0.570316" origin_rpy="0 0 0"
     material_name="white"
-    inertia_origin_xyz="-0.001 -0.0211 0.0" inertia_origin_rpy="0 0 0"
-    mass="0.2"
-    ixx="1e-4" iyy="1e-4" izz="1e-4" ixy="-0.0" iyz="0.0" ixz="0.0"
+    inertia_origin_xyz="0.0036112727264542635 -0.014760653808445767 -0.00103677815369696" inertia_origin_rpy="0 0 0"
+    mass="0.5810486809925093"
+    ixx="0.000385" iyy="0.000495" izz="0.000263" ixy="1e-05" iyz="-2e-06" ixz="3e-06"
   />
   <xacro:arctos_link
     name="Left_jaw_1"
-    origin_xyz="0.0 0.323 -0.5685" origin_rpy="0 0 0"
+    origin_xyz="-0.007934 0.359845 -0.599867" origin_rpy="0 0 0"
     material_name="white"
-    inertia_origin_xyz="-0.0 -0.0211 0.0" inertia_origin_rpy="0 0 0"
-    mass="0."
-    ixx="0.0" iyy="0.0" izz="0.0" ixy="-0.0" iyz="0.0" ixz="0.0"
+    inertia_origin_xyz="-0.011142702480351952 -0.009692440309284511 -0.009385792627785827" inertia_origin_rpy="0 0 0"
+    mass="0.07369602565859415"
+    ixx="1.1e-05" iyy="6e-06" izz="1.4e-05" ixy="2e-06" iyz="-0.0" ixz="-0.0"
   />
   <xacro:arctos_link
     name="Right_jaw_1"
-    origin_xyz="0.0 0.323 -0.5685" origin_rpy="0 0 0"
+    origin_xyz="-0.007934 0.359845 -0.539867" origin_rpy="0 0 0"
     material_name="white"
-    inertia_origin_xyz="-0.001 -0.0211 0.0" inertia_origin_rpy="0 0 0"
-    mass="0."
-    ixx="0.0" iyy="0.0" izz="0.0" ixy="-0.0" iyz="0.0" ixz="0.0"
+    inertia_origin_xyz="-0.008289104952972526 -0.009768535307719373 0.009395511902715814" inertia_origin_rpy="0 0 0"
+    mass="0.07312902168719511"
+    ixx="1.1e-05" iyy="6e-06" izz="1.4e-05" ixy="-1e-06" iyz="0.0" ixz="-1e-06"
   />
   <!-- Fixed gripper joint, no axis needed -->
@@ -32,5 +32,5 @@
     name="Gripper_joint" type="fixed"
     parent="Link_6_1" child="Gripper_1"
-    origin_xyz="0.0 -0.0 0.0" origin_rpy="0 0 0"
+    origin_xyz="0.0 -0.006085 0.0" origin_rpy="0 0 0"
     limit_u="0.0" limit_l="0.0" limit_e="0.0" limit_v="0.0"
   />
@@ -38,28 +38,14 @@
   <!-- TODO: Movement inverted -->
   <xacro:arctos_joint
-    name="Left_jaw_joint"
-    type="prismatic"
-    parent="Gripper_1"
-    child="Left_jaw_1"
-    origin_xyz="0.0 0.0 0.0"
-    origin_rpy="0 0 0"
-    axis_xyz="0 0 1"
-    limit_u="0.015"
-    limit_l="0.0"
-    limit_e="1.0"
-    limit_v="10.0"
+    name="Left_jaw_joint" type="prismatic"
+    parent="Gripper_1" child="Left_jaw_1"
+    origin_xyz="0.007741 -0.039998 0.029551" origin_rpy="0 0 0" axis_xyz="-0.0 0.0 -1.0"
+    limit_u="0.015" limit_l="0.0" limit_e="100.0" limit_v="100.0"
   />
   <xacro:arctos_joint
-    name="Right_jaw_joint"
-    type="prismatic"
-    parent="Gripper_1"
-    child="Right_jaw_1"
-    origin_xyz="0.0 0.0 0.0"
-    origin_rpy="0 0 0"
-    axis_xyz="0 0 1"
-    limit_u="0.015"
-    limit_l="0.0"
-    limit_e="1.0"
-    limit_v="10.0"
+    name="Right_jaw_joint" type="prismatic"
+    parent="Gripper_1" child="Right_jaw_1"
+    origin_xyz="0.007741 -0.039998 -0.030449" origin_rpy="0 0 0" axis_xyz="0.0 -0.0 1.0"
+    limit_u="0.015" limit_l="0.0" limit_e="100.0" limit_v="100.0"
   />
 </robot>

File: arctos_description/urdf/arctos_ros2_control.xacro (robot description, xacro)
@@ -7,5 +7,5 @@
         <plugin>arctos_interface/ArctosInterface</plugin>
       </hardware>
-      <xacro:arctos_control
+      <!-- <xacro:arctos_control
         name="X_joint"
         limit_u="${pi}" limit_l="${-pi}"
@@ -18,9 +18,51 @@
         name="Z_joint"
         limit_u="0.65" limit_l="-1.6"
-      />
+      /> -->
+       <joint name="X_joint">
+        <command_interface name="position">
+          <param name="min">{-pi}</param>
+          <param name="max">{pi}</param>
+        </command_interface>
+        <command_interface name="velocity">
+          <param name="min">-3.15</param>
+          <param name="max">3.15</param>
+        </command_interface>
+        <state_interface name="position">
+          <param name="initial_value">0.0</param>
+        </state_interface>
+        <state_interface name="velocity" />
+      </joint>
+      <joint name="Y_joint">
+        <command_interface name="position">
+          <param name="min">{-0.96}</param>
+          <param name="max">{2.18}</param>
+        </command_interface>
+        <command_interface name="velocity">
+          <param name="min">-3.15</param>
+          <param name="max">3.15</param>
+        </command_interface>
+        <state_interface name="position">
+          <param name="initial_value">0.0</param>
+        </state_interface>
+        <state_interface name="velocity" />
+      </joint>
+      <joint name="Z_joint">
+        <command_interface name="position">
+          <param name="min">{-pi/2}</param>
+          <param name="max">{55/180*pi}</param>
+        </command_interface>
+        <command_interface name="velocity">
+          <param name="min">-3.15</param>
+          <param name="max">3.15</param>
+        </command_interface>
+        <state_interface name="position">
+          <param name="initial_value">0.0</param>
+        </state_interface>
+        <state_interface name="velocity" />
+      </joint>
       <joint name="A_joint">
         <command_interface name="position">
-          <param name="min">{-2*pi}</param>
-          <param name="max">{2*pi}</param>
+          <param name="min">{-pi/2}</param>
+          <param name="max">{pi/2}</param>
         </command_interface>
         <command_interface name="velocity">
@@ -35,6 +77,6 @@
       <joint name="B_joint">
         <command_interface name="position">
-          <param name="min">{-2*pi}</param>
-          <param name="max">{2*pi}</param>
+          <param name="min">{-1.55}</param>
+          <param name="max">{1.55}</param>
         </command_interface>
         <command_interface name="velocity">
@@ -49,6 +91,6 @@
       <joint name="C_joint">
         <command_interface name="position">
-          <param name="min">{-2*pi}</param>
-          <param name="max">{2*pi}</param>
+          <param name="min">{-pi}</param>
+          <param name="max">{pi}</param>
         </command_interface>
         <command_interface name="velocity">
