Commit message: replace arctos model with Denso model

File: arctos_description/urdf/arctos.xacro (robot description, xacro)
@@ -3,5 +3,5 @@
   <xacro:include filename="$(find arctos_description)/urdf/common/materials.xacro" />
   <xacro:include filename="$(find arctos_description)/urdf/common/joint_link.xacro" />
-  <xacro:include filename="$(find arctos_description)/urdf/arctos_gripper.xacro" />
+  <!-- <xacro:include filename="$(find arctos_description)/urdf/arctos_gripper.xacro" /> -->
   <link name="world" />
   <joint name="world_joint" type="fixed">
@@ -12,105 +12,100 @@
   <xacro:arctos_link
     name="base_link"
+    inertia_origin_xyz="-0.00047006 -0.012257 0.10022" inertia_origin_rpy="0 0 0"
+    mass="55.785"
+    ixx="0.39179" ixy="-0.0027323" ixz="-0.00075955" iyy="0.323" iyz="-0.022558" izz="0.34492"
     origin_xyz="0 0 0" origin_rpy="0 0 0"
-    material_name="white"
-    inertia_origin_xyz="0.0009375030874740357 0.047087016508753216 0.06663230338123677"
-    inertia_origin_rpy="0 0 0"
-    mass="2.3"
-    ixx="0.0143" iyy="0.0055" izz="0.015" ixy="0.0" iyz="0.0" ixz="0.0"
+    material_name="base_blue"
   />
   <xacro:arctos_link
-    name="Link_1_1"
-    origin_xyz="-0.0 -0.000 -0.1126" origin_rpy="0 0 0"
-    material_name="white"
-    inertia_origin_xyz="-0.0088 -0.0005 ${0.2116-0.1126}" inertia_origin_rpy="0 0 0"
-    mass="3.0396"
-    ixx="0.0143" iyy="${0.0168*0.96536}" izz="${0.0084*0.96082}" ixy="${0.0143*-0.03956}"
-    ixz="${0.0143*-0.11546}" iyz="${0.0168*0.25198}"
+    name="link_1"
+    inertia_origin_xyz="0.0075871 0.03734 0.10645" inertia_origin_rpy="0 0 0"
+    mass="44.267"
+    ixx="0.28548" ixy="-0.012987" ixz="-0.013929" iyy="0.25047" iyz="-0.073189" izz="0.26167"
+    origin_xyz="0 0 0" origin_rpy="0 0 0"
+    material_name="blue"
   />
   <xacro:arctos_link
-    name="Link_2_1"
-    origin_xyz="0.0 0.020356 -0.2876" origin_rpy="0 0 0"
-    material_name="white"
-    inertia_origin_xyz="0.0042 ${-0.0098+0.020356} ${0.4174-0.2876}" inertia_origin_rpy="0 0 0"
-    mass="2.527"
-    ixx="${0.0282*0.99851}" iyy="${0.03*0.99865}" izz="${0.0063*0.99982}" ixy="${0.0282*0.05146}"
-    iyz="${0.03*-0.00591}" ixz="${0.0282*-0.01813}"
+    name="link_2"
+    inertia_origin_xyz="-0.068044 0.021826 0.15762" inertia_origin_rpy="0 0 0"
+    mass="43.339"
+    ixx="0.97722" ixy="0.00042244" ixz="-0.021124" iyy="0.93504" iyz="-0.078229" izz="0.099171"
+    origin_xyz="0 0 0" origin_rpy="0 0 0"
+    material_name="gray"
   />
   <xacro:arctos_link
-    name="Link_3_1"
-    origin_xyz="-0.0 0.019045 -0.54864" origin_rpy="0 0 0"
-    material_name="white"
-    inertia_origin_xyz="0.00158 -0.053 0.009" inertia_origin_rpy="0 0 0"
-    mass="0.87"
-    ixx="${0.0028*0.99944}" iyy="${0.0011*0.98426}" izz="${0.0027*0.98428}" ixy="${0.0028*-0.02203}"
-    iyz="${0.001*-0.17481}" ixz="${0.0028*0.02507}"
+    name="link_3"
+    inertia_origin_xyz="0.054747 0.060447 0.045778" inertia_origin_rpy="0 0 0"
+    mass="37.594"
+    ixx="0.31727" ixy="0.0065087" ixz="0.0048815" iyy="0.16116" iyz="-0.088578" izz="0.26582"
+    origin_xyz="0 0 0" origin_rpy="0 0 0"
+    material_name="gray"
   />
   <xacro:arctos_link
-    name="Link_4_1"
-    origin_xyz="0.0 0.1578 -0.5704" origin_rpy="0 0 0"
-    material_name="white"
-    inertia_origin_xyz="0.0 -0.0535 -0.001733" inertia_origin_rpy="0 0 0"
+    name="link_4"
+    inertia_origin_xyz="0.0051846 0.10645 0.00064606" inertia_origin_rpy="0 0 0"
     mass="1.006"
-    ixx="${0.0021*0.99726}" iyy="${0.0024*0.99801}" izz="${0.0032*0.99925}" ixy="${0.0021*-0.6305}"
-    iyz="${0.0024*0.00082}" ixz="${0.0021*0.03862}"
+    ixx="0.062769" ixy="-0.001868" ixz="-3.6977E-05" iyy="0.028683" iyz="0.00032273" izz="0.069443"
+    origin_xyz="0 0 0" origin_rpy="0 0 0"
+    material_name="gray"
   />
   <xacro:arctos_link
-    name="Link_5_1"
-    origin_xyz="0.0 0.2832 -0.56856" origin_rpy="0 0 0"
-    material_name="white"
-    inertia_origin_xyz="-0.0007 -0.0142 -0.0008" inertia_origin_rpy="0 0 0"
-    mass="0.3344"
-    ixx="0.0002" iyy="0.0005" izz="0.0005" ixy="0.0" iyz="0.0" ixz="0.0"
+    name="link_5"
+    inertia_origin_xyz="-0.00049422 0.0067098 -2.4246E-07" inertia_origin_rpy="0 0 0"
+    mass="0.34309"
+    ixx="0.00034995" ixy="-1.1371E-06" ixz="1.2487E-09" iyy="0.00022745" iyz="1.4302E-09" izz="0.00030039"
+    origin_xyz="0 0 0" origin_rpy="0 0 0"
+    material_name="gray"
   />
   <xacro:arctos_link
-    name="Link_6_1"
-    origin_xyz="0.0 0.323 -0.5685" origin_rpy="0 0 0"
-    material_name="white"
-    inertia_origin_xyz="-0.0 -0.0 0.0" inertia_origin_rpy="0.0 0.0 0.0"
-    mass="1e-3"
-    ixx="1e-3" iyy="1e-3" izz="1e-3" ixy="-0.0" iyz="0.0" ixz="0.0"
+    name="link_6"
+    inertia_origin_xyz="3.1972E-05 0.011587 0" inertia_origin_rpy="0.0 0.0 0.0"
+    mass="0.068739"
+    ixx="2.0617E-05" ixy="-2.849E-08" ixz="-7.3853E-22" iyy="3.4376E-05" iyz="2.1018E-21" izz="2.0453E-05"
+    origin_xyz="0 0 0" origin_rpy="0 0 0"
+    material_name="gray"
   />
   <!--Change limit of joints here-->
   <xacro:arctos_joint
     name="X_joint" type="revolute"
-    parent="base_link" child="Link_1_1"
-    origin_xyz="0.0 0.0 0.1126" origin_rpy="0 0 0"
-    axis_xyz="0.0 0.0 1.0"
-    limit_u="${pi}" limit_l="${-pi}" limit_e="24.3" limit_v="15.0" mimic=""
+    parent="base_link" child="link_1"
+    origin_xyz="0 0 0.183" origin_rpy="0 0 0"
+    axis_xyz="0 0 1"
+    limit_l="-2.9671" limit_u="2.9671"  limit_e="1" limit_v="3.0543" mimic=""
   />
   <xacro:arctos_joint
     name="Y_joint" type="revolute"
-    parent="Link_1_1" child="Link_2_1"
-    origin_xyz="0.0 -0.020356 ${0.2876-0.1126}" origin_rpy="0 0 0"
-    axis_xyz="1.0 -0.0 -0.0"
-    limit_u="2.18" limit_l="-0.96" limit_e="270.0" limit_v="1.4" mimic=""
+    parent="link_1" child="link_2"
+    origin_xyz="-0.048 0.075 0.15" origin_rpy="0 0 0"
+    axis_xyz="-1 0 0"
+    limit_l="-1.7453" limit_u="2.3562" limit_e="1" limit_v="3.4907" mimic=""
   />
   <xacro:arctos_joint
     name="Z_joint" type="revolute"
-    parent="Link_2_1" child="Link_3_1"
-    origin_xyz="0.0 0.001365 0.261035" origin_rpy="0 0 0"
-    axis_xyz="1.0 -0.0 0.0"
-    limit_u="${55/180*pi}" limit_l="${-pi/2}" limit_e="97.0" limit_v="1.4" mimic=""
+    parent="link_2" child="link_3"
+    origin_xyz="0 0.029976 0.36377" origin_rpy="0 0 0"
+    axis_xyz="-1 0 0"
+    limit_l="-2.0769" limit_u="2.9496" limit_e="1" limit_v="3.4907" mimic=""
   />
   <xacro:arctos_joint
     name="A_joint" type="revolute"
-    parent="Link_3_1" child="Link_4_1"
-    origin_xyz="0 -0.13881 0.0217651" origin_rpy="0 0 0"
+    parent="link_3" child="link_4"
+    origin_xyz="0.048 0.198 0.09" origin_rpy="0 0 0"
     axis_xyz="0.0 1.0 0.0"
-    limit_u="${pi/2}" limit_l="${-pi/2}" limit_e="22.0" limit_v="4.4" mimic=""
+    limit_l="-3.3161" limit_u="3.3161" limit_e="1" limit_v="5.236" mimic=""
   />
   <xacro:arctos_joint
     name="B_joint" type="revolute"
-    parent="Link_4_1" child="Link_5_1"
-    origin_xyz="0.0 -0.12543 -0.00184" origin_rpy="0 0 0"
-    axis_xyz="-1.0 0.0 0.0"
-    limit_u="1.55" limit_l="-1.55" limit_e="16.0" limit_v="3.0" mimic=""
+    parent="link_4" child="link_5"
+    origin_xyz="0 0.207 0" origin_rpy="0 0 0"
+    axis_xyz="1 0 0"
+    limit_l="-2.0944" limit_u="2.0944" limit_e="1" limit_v="5.236" mimic=""
   />
   <xacro:arctos_joint
     name="C_joint" type="revolute"
-    parent="Link_5_1" child="Link_6_1"
-    origin_xyz="0.0 -0.0398 0.0" origin_rpy="0 0 0"
+    parent="link_5" child="link_6"
+    origin_xyz="0 0.052 0" origin_rpy="0 0 0"
     axis_xyz="0.0 1.0 0.0"
-    limit_u="${pi}" limit_l="${-pi}" limit_e="16.0" limit_v="3.0" mimic=""
+    limit_l="-6.2832" limit_u="6.2832" limit_e="1" limit_v="8.3776" mimic=""
   />
 </robot>

File: arctos_description/urdf/common/joint_link.xacro (robot description, xacro)
@@ -8,5 +8,5 @@
         <origin xyz="${origin_xyz}" rpy="${origin_rpy}" />
         <geometry>
-          <mesh filename="package://arctos_description/meshes/${name}.stl" scale="0.001 0.001 0.001" />
+          <mesh filename="package://arctos_description/meshes/${name}.STL"/>
         </geometry>
         <material name="${material_name}" />
@@ -15,5 +15,5 @@
         <origin xyz="${origin_xyz}" rpy="${origin_rpy}" />
         <geometry>
-          <mesh filename="package://arctos_description/meshes/${name}.stl" scale="0.001 0.001 0.001" />
+          <mesh filename="package://arctos_description/meshes/${name}.STL"/>
         </geometry>
       </collision>

File: arctos_description/urdf/common/materials.xacro (robot description, xacro)
@@ -7,3 +7,12 @@
     <color rgba="0.0 0.0 0.0 1.0" />
   </material>
+  <material name="base_blue">
+    <color rgba="0.50196 0.50196 1 1" />
+  </material>
+  <material name="blue">
+    <color rgba="0.78431 0.98039 0.98039 1" />
+  </material>
+  <material name="gray">
+    <color rgba="0.78431 0.98039 0.98039 1" />
+  </material>
 </robot>

Commit message: 1st-steop: update to denso_moveit_config: make it run normally on bringup.

File: arctos_description/urdf/arctos.xacro (robot description, xacro)
@@ -86,5 +86,5 @@
     origin_xyz="0 0.029976 0.36377" origin_rpy="0 0 0"
     axis_xyz="-1 0 0"
-    limit_l="-2.0769" limit_u="2.9496" limit_e="1" limit_v="3.4907" mimic=""
+    limit_l="-2.0769" limit_u="1.5" limit_e="1" limit_v="3.4907" mimic=""
   />
   <xacro:arctos_joint

File: arctos_moveit_config/config/arctos.ros2_control.xacro (robot description, xacro)
@@ -1,5 +1,5 @@
 <?xml version="1.0"?>
 <robot xmlns:xacro="http://www.ros.org/wiki/xacro">
-  <xacro:macro name="arctos_ros2_control" params="name initial_positions_file">
+  <xacro:macro name="arctos_ros2_control" params="name initial_positions_file sim:=false">
     <!--xacro.load_yaml must be used instead of load_yaml, or else we gonna get error: Using load_yaml() directly is deprecated. Use xacro.load_yaml() instead.-->
     <xacro:property name="initial_positions"
@@ -7,18 +7,20 @@
     <ros2_control name="${name}" type="system">
       <hardware>
-        <plugin>arctos_interface/ArctosInterface</plugin>
+        <!-- By default, set up controllers for simulation. This won't work on real hardware -->
+        <xacro:if value="${sim}">
+          <plugin>mock_components/GenericSystem</plugin>
+        </xacro:if>
+        <xacro:unless value="${sim}">
+          <plugin>arctos_interface/ArctosInterface</plugin>
+        </xacro:unless>
       </hardware>
-      <!-- <hardware> -->
-      <!-- By default, set up controllers for simulation. This won't work on real hardware -->
-      <!-- <plugin>mock_components/GenericSystem</plugin> -->
-      <!-- </hardware> -->
       <joint name="X_joint">
         <command_interface name="position">
-          <param name="min">{-pi}</param>
-          <param name="max">{pi}</param>
+          <param name="min">-2.967060</param>
+          <param name="max">2.967060</param>
         </command_interface>
         <command_interface name="velocity">
-          <param name="min">-3.15</param>
-          <param name="max">3.15</param>
+          <param name="min">0</param>
+          <param name="max">0.392699081698724</param>
         </command_interface>
         <state_interface name="position">
@@ -29,10 +31,10 @@
       <joint name="Y_joint">
         <command_interface name="position">
-          <param name="min">{-0.96}</param>
-          <param name="max">{2.18}</param>
+          <param name="min">-2.094395</param>
+          <param name="max">2.094395</param>
         </command_interface>
         <command_interface name="velocity">
-          <param name="min">-3.15</param>
-          <param name="max">3.15</param>
+          <param name="min">0</param>
+          <param name="max">0.261799387799149</param>
         </command_interface>
         <state_interface name="position">
@@ -43,10 +45,10 @@
       <joint name="Z_joint">
         <command_interface name="position">
-          <param name="min">{-pi/2}</param>
-          <param name="max">{55/180*pi}</param>
+          <param name="min">-2.0769</param>
+          <param name="max">1.5</param>
         </command_interface>
         <command_interface name="velocity">
-          <param name="min">-3.15</param>
-          <param name="max">3.15</param>
+          <param name="min">0</param>
+          <param name="max">0.285832571599111</param>
         </command_interface>
         <state_interface name="position">
@@ -57,10 +59,10 @@
       <joint name="A_joint">
         <command_interface name="position">
-          <param name="min">{-pi/2}</param>
-          <param name="max">{pi/2}</param>
+          <param name="min">-3.3161</param>
+          <param name="max">3.3161</param>
         </command_interface>
         <command_interface name="velocity">
-          <param name="min">-3.2</param>
-          <param name="max">3.2</param>
+          <param name="min">0</param>
+          <param name="max">0.392699081698724</param>
         </command_interface>
         <state_interface name="position">
@@ -71,10 +73,10 @@
       <joint name="B_joint">
         <command_interface name="position">
-          <param name="min">{-1.55}</param>
-          <param name="max">{1.55}</param>
+          <param name="min">-2.0944</param>
+          <param name="max">2.0944</param>
         </command_interface>
         <command_interface name="velocity">
-          <param name="min">-3.2</param>
-          <param name="max">3.2</param>
+          <param name="min">0</param>
+          <param name="max">0.302168853397778</param>
         </command_interface>
         <state_interface name="position">
@@ -85,10 +87,10 @@
       <joint name="C_joint">
         <command_interface name="position">
-          <param name="min">{-pi}</param>
-          <param name="max">{pi}</param>
+          <param name="min">-6.283185</param>
+          <param name="max">6.283185</param>
         </command_interface>
         <command_interface name="velocity">
-          <param name="min">-3.2</param>
-          <param name="max">3.2</param>
+          <param name="min">0</param>
+          <param name="max">0.628318530717959</param>
         </command_interface>
         <state_interface name="position">
@@ -97,22 +99,4 @@
         <state_interface name="velocity" />
       </joint>
-      <joint name="Left_jaw_joint">
-        <command_interface name="position" />
-        <param name="min">{0}</param>
-        <param name="max">{0.015}</param>
-        <command_interface name="velocity" />
-        <state_interface name="position">
-          <param name="initial_value">${initial_positions['Left_jaw_joint']}</param>
-        </state_interface>
-        <state_interface name="velocity" />
-      </joint>
-      <!-- <sensor name="tcp_fts_sensor">
-        <state_interface name="force.x"/>
-        <state_interface name="force.y"/>
-        <state_interface name="force.z"/>
-        <state_interface name="torque.x"/>
-        <state_interface name="torque.y"/>
-        <state_interface name="torque.z"/>
-      </sensor> -->
     </ros2_control>
   </xacro:macro>

File: arctos_moveit_config/config/arctos.urdf.xacro (robot description, xacro)
@@ -3,7 +3,7 @@
     <xacro:arg name="initial_positions_file" default="initial_positions.yaml" />
     <!-- Import arctos urdf file -->
-    <xacro:include filename="$(find arctos_description)/urdf/arctos.xacro" />
+    <xacro:include filename="$(find arctos_description)/urdf/arctos.urdf" />
     <!-- Import control_xacro -->
     <xacro:include filename="arctos.ros2_control.xacro" />
-    <xacro:arctos_ros2_control name="RealSystems" initial_positions_file="$(arg initial_positions_file)"/>
+    <xacro:arctos_ros2_control name="RealSystem" initial_positions_file="$(arg initial_positions_file)" sim="false"/>
 </robot>
