Commit message: Big cleanup, remove xyz, remove config in description folder

File: arctos_description/urdf/arctos.urdf (robot description, URDF)
Before this commit: robot arctos, 11 links, 10 joints
Joints:
- joint Right_jaw_joint: mimic (none) -> joint=Left_jaw_joint

File: arctos_description/urdf/arctos.xacro (robot description, xacro)
@@ -3,5 +3,4 @@
   <xacro:include filename="$(find arctos_description)/urdf/common/materials.xacro" />
   <xacro:include filename="$(find arctos_description)/urdf/common/joint_link.xacro" />
-  <xacro:include filename="$(find arctos_description)/urdf/arctos_ros2_control.xacro" />
   <xacro:include filename="$(find arctos_description)/urdf/arctos_gripper.xacro" />
   <link name="world" />
@@ -78,5 +77,5 @@
     origin_xyz="0.0 0.0 0.1126" origin_rpy="0 0 0"
     axis_xyz="0.0 0.0 1.0"
-    limit_u="${pi}" limit_l="${-pi}" limit_e="24.3" limit_v="15.0"
+    limit_u="${pi}" limit_l="${-pi}" limit_e="24.3" limit_v="15.0" mimic=""
   />
   <xacro:arctos_joint
@@ -85,5 +84,5 @@
     origin_xyz="0.0 -0.020356 ${0.2876-0.1126}" origin_rpy="0 0 0"
     axis_xyz="1.0 -0.0 -0.0"
-    limit_u="2.18" limit_l="-0.96" limit_e="270.0" limit_v="1.4"
+    limit_u="2.18" limit_l="-0.96" limit_e="270.0" limit_v="1.4" mimic=""
   />
   <xacro:arctos_joint
@@ -92,5 +91,5 @@
     origin_xyz="0.0 0.001365 0.261035" origin_rpy="0 0 0"
     axis_xyz="1.0 -0.0 0.0"
-    limit_u="${55/180*pi}" limit_l="${-pi/2}" limit_e="97.0" limit_v="1.4"
+    limit_u="${55/180*pi}" limit_l="${-pi/2}" limit_e="97.0" limit_v="1.4" mimic=""
   />
   <xacro:arctos_joint
@@ -99,5 +98,5 @@
     origin_xyz="0 -0.13881 0.0217651" origin_rpy="0 0 0"
     axis_xyz="0.0 1.0 0.0"
-    limit_u="${pi/2}" limit_l="${-pi/2}" limit_e="22.0" limit_v="4.4"
+    limit_u="${pi/2}" limit_l="${-pi/2}" limit_e="22.0" limit_v="4.4" mimic=""
   />
   <xacro:arctos_joint
@@ -106,5 +105,5 @@
     origin_xyz="0.0 -0.12543 -0.00184" origin_rpy="0 0 0"
     axis_xyz="-1.0 0.0 0.0"
-    limit_u="1.55" limit_l="-1.55" limit_e="16.0" limit_v="3.0"
+    limit_u="1.55" limit_l="-1.55" limit_e="16.0" limit_v="3.0" mimic=""
   />
   <xacro:arctos_joint
@@ -113,6 +112,5 @@
     origin_xyz="0.0 -0.0398 0.0" origin_rpy="0 0 0"
     axis_xyz="0.0 1.0 0.0"
-    limit_u="${pi}" limit_l="${-pi}" limit_e="16.0" limit_v="3.0"
+    limit_u="${pi}" limit_l="${-pi}" limit_e="16.0" limit_v="3.0" mimic=""
   />
-  <xacro:arctos_ros2_control name="arctos_interface" />
 </robot>

File: arctos_description/urdf/arctos_gripper.xacro (robot description, xacro)
@@ -33,5 +33,5 @@
     parent="Link_6_1" child="Gripper_1"
     origin_xyz="0.0 -0.006085 0.0" origin_rpy="0 0 0"
-    limit_u="0.0" limit_l="0.0" limit_e="0.0" limit_v="0.0"
+    limit_u="0.0" limit_l="0.0" limit_e="0.0" limit_v="0.0" mimic=""
   />
   <!-- Left jaw joint, prismatic with axis directly defined -->
@@ -41,5 +41,5 @@
     parent="Gripper_1" child="Left_jaw_1"
     origin_xyz="0.007741 -0.039998 0.029551" origin_rpy="0 0 0" axis_xyz="-0.0 0.0 -1.0"
-    limit_u="0.015" limit_l="0.0" limit_e="100.0" limit_v="100.0"
+    limit_u="0.015" limit_l="0.0" limit_e="100.0" limit_v="100.0" mimic=""
   />
   <xacro:arctos_joint
@@ -47,5 +47,5 @@
     parent="Gripper_1" child="Right_jaw_1"
     origin_xyz="0.007741 -0.039998 -0.030449" origin_rpy="0 0 0" axis_xyz="0.0 -0.0 1.0"
-    limit_u="0.015" limit_l="0.0" limit_e="100.0" limit_v="100.0"
+    limit_u="0.015" limit_l="0.0" limit_e="100.0" limit_v="100.0" mimic="Left_jaw_joint"
   />
 </robot>

File: arctos_description/urdf/common/joint_link.xacro (robot description, xacro)
@@ -28,5 +28,5 @@
   <!-- TODO: Add param for mechanicalReduction -->
   <xacro:macro name="arctos_joint"
-    params="name type parent child origin_xyz origin_rpy axis_xyz='0 0 0' limit_u limit_l limit_e limit_v">
+    params="name type parent child origin_xyz origin_rpy axis_xyz='0 0 0' limit_u limit_l limit_e limit_v mimic">
     <joint name="${name}" type="${type}">
       <parent link="${parent}" />
@@ -35,4 +35,7 @@
       <axis xyz="${axis_xyz}" />
       <limit upper="${limit_u}" lower="${limit_l}" effort="${limit_e}" velocity="${limit_v}" />
+      <xacro:if value="${mimic != ''}">
+          <mimic joint="${mimic}" />
+      </xacro:if>
     </joint>
     <!-- Add transmission element -->

File: arctos_moveit_config/config/arctos.ros2_control.xacro (robot description, xacro)
@@ -2,18 +2,23 @@
 <robot xmlns:xacro="http://www.ros.org/wiki/xacro">
   <xacro:macro name="arctos_ros2_control" params="name initial_positions_file">
+    <!--xacro.load_yaml must be used instead of load_yaml, or else we gonna get error: Using load_yaml() directly is deprecated. Use xacro.load_yaml() instead.-->
     <xacro:property name="initial_positions"
-      value="${load_yaml(initial_positions_file)['initial_positions']}" />
+      value="${xacro.load_yaml(initial_positions_file)['initial_positions']}" />
     <ros2_control name="${name}" type="system">
       <hardware>
         <plugin>arctos_interface/ArctosInterface</plugin>
       </hardware>
+      <!-- <hardware> -->
+      <!-- By default, set up controllers for simulation. This won't work on real hardware -->
+      <!-- <plugin>mock_components/GenericSystem</plugin> -->
+      <!-- </hardware> -->
       <joint name="X_joint">
         <command_interface name="position">
-          <!-- <param name="min">{-2*pi}</param>
-          <param name="max">{2*pi}</param> -->
+          <param name="min">{-pi}</param>
+          <param name="max">{pi}</param>
         </command_interface>
         <command_interface name="velocity">
-          <!-- <param name="min">-3.15</param>
-          <param name="max">3.15</param> -->
+          <param name="min">-3.15</param>
+          <param name="max">3.15</param>
         </command_interface>
         <state_interface name="position">
@@ -24,10 +29,10 @@
       <joint name="Y_joint">
         <command_interface name="position">
-          <!-- <param name="min">{-2*pi}</param>
-          <param name="max">{2*pi}</param> -->
+          <param name="min">{-0.96}</param>
+          <param name="max">{2.18}</param>
         </command_interface>
         <command_interface name="velocity">
-          <!-- <param name="min">-3.15</param>
-          <param name="max">3.15</param> -->
+          <param name="min">-3.15</param>
+          <param name="max">3.15</param>
         </command_interface>
         <state_interface name="position">
@@ -38,10 +43,10 @@
       <joint name="Z_joint">
         <command_interface name="position">
-          <!-- <param name="min">{-pi}</param>
-          <param name="max">{pi}</param> -->
+          <param name="min">{-pi/2}</param>
+          <param name="max">{55/180*pi}</param>
         </command_interface>
         <command_interface name="velocity">
-          <!-- <param name="min">-3.15</param>
-          <param name="max">3.15</param> -->
+          <param name="min">-3.15</param>
+          <param name="max">3.15</param>
         </command_interface>
         <state_interface name="position">
@@ -52,10 +57,10 @@
       <joint name="A_joint">
         <command_interface name="position">
-          <!-- <param name="min">{-2*pi}</param>
-          <param name="max">{2*pi}</param> -->
+          <param name="min">{-pi/2}</param>
+          <param name="max">{pi/2}</param>
         </command_interface>
         <command_interface name="velocity">
-          <!-- <param name="min">-3.2</param>
-          <param name="max">3.2</param> -->
+          <param name="min">-3.2</param>
+          <param name="max">3.2</param>
         </command_interface>
         <state_interface name="position">
@@ -66,10 +71,10 @@
       <joint name="B_joint">
         <command_interface name="position">
-          <!-- <param name="min">{-2*pi}</param>
-          <param name="max">{2*pi}</param> -->
+          <param name="min">{-1.55}</param>
+          <param name="max">{1.55}</param>
         </command_interface>
         <command_interface name="velocity">
-          <!-- <param name="min">-3.2</param>
-          <param name="max">3.2</param> -->
+          <param name="min">-3.2</param>
+          <param name="max">3.2</param>
         </command_interface>
         <state_interface name="position">
@@ -80,10 +85,10 @@
       <joint name="C_joint">
         <command_interface name="position">
-          <!-- <param name="min">{-2*pi}</param>
-          <param name="max">{2*pi}</param> -->
+          <param name="min">{-pi}</param>
+          <param name="max">{pi}</param>
         </command_interface>
         <command_interface name="velocity">
-          <!-- <param name="min">-3.2</param>
-          <param name="max">3.2</param> -->
+          <param name="min">-3.2</param>
+          <param name="max">3.2</param>
         </command_interface>
         <state_interface name="position">
@@ -94,4 +99,6 @@
       <joint name="Left_jaw_joint">
         <command_interface name="position" />
+        <param name="min">{0}</param>
+        <param name="max">{0.015}</param>
         <command_interface name="velocity" />
         <state_interface name="position">
@@ -100,12 +107,12 @@
         <state_interface name="velocity" />
       </joint>
-      <joint name="Right_jaw_joint">
-        <command_interface name="position" />
-        <command_interface name="velocity" />
-        <state_interface name="position">
-          <param name="initial_value">${initial_positions['Right_jaw_joint']}</param>
-        </state_interface>
-        <state_interface name="velocity" />
-      </joint>
+      <!-- <sensor name="tcp_fts_sensor">
+        <state_interface name="force.x"/>
+        <state_interface name="force.y"/>
+        <state_interface name="force.z"/>
+        <state_interface name="torque.x"/>
+        <state_interface name="torque.y"/>
+        <state_interface name="torque.z"/>
+      </sensor> -->
     </ros2_control>
   </xacro:macro>

File: arctos_moveit_config/config/arctos.urdf.xacro (robot description, xacro)
@@ -3,7 +3,7 @@
     <xacro:arg name="initial_positions_file" default="initial_positions.yaml" />
     <!-- Import arctos urdf file -->
-    <xacro:include filename="$(find arctos_description)/urdf/arctos.urdf" />
+    <xacro:include filename="$(find arctos_description)/urdf/arctos.xacro" />
     <!-- Import control_xacro -->
     <xacro:include filename="arctos.ros2_control.xacro" />
-    <!-- <xacro:arctos_ros2_control name="FakeSystem" initial_positions_file="$(arg initial_positions_file)"/> -->
+    <xacro:arctos_ros2_control name="RealSystems" initial_positions_file="$(arg initial_positions_file)"/>
 </robot>

Commit message: Update

File: arctos_description/urdf/arctos.urdf (robot description, URDF)
Before this commit: robot arctos, 8 links, 7 joints
Links:
- link link_4: mass 1.006 -> 14.917
Joints:
- joint A_joint: axis 0.0 1.0 0.0 -> 0 0 1; origin xyz=0.048 0.198 0.09 rpy=0 0 0 -> xyz=0.048 -0.09 0.198 rpy=0 0 0
- joint B_joint: origin xyz=0 0.207 0 rpy=0 0 0 -> xyz=0 0 0.207 rpy=0 0 0
- joint C_joint: axis 0.0 1.0 0.0 -> 0.0 0.0 1.0; origin xyz=0 0.052 0 rpy=0 0 0 -> xyz=0 0 0.052 rpy=0 0 0
- joint Z_joint: limit lower=-2.0769 upper=2.9496 effort=1 velocity=3.4907 -> lower=-2.0769 upper=2.949606436 effort=1 velocity=3.4907

File: arctos_description/urdf/arctos.xacro (robot description, xacro)
@@ -36,7 +36,7 @@
   <xacro:arctos_link
     name="link_3"
-    inertia_origin_xyz="0.054747 0.060447 0.045778" inertia_origin_rpy="0 0 0"
+    inertia_origin_xyz="0.054747 -0.045778 0.060447" inertia_origin_rpy="0 0 0"
     mass="37.594"
-    ixx="0.31727" ixy="0.0065087" ixz="0.0048815" iyy="0.16116" iyz="-0.088578" izz="0.26582"
+    ixx="0.31727" ixy="-0.0048815" ixz="0.0065087" iyy="0.26582" iyz="0.088578" izz="0.16116"
     origin_xyz="0 0 0" origin_rpy="0 0 0"
     material_name="gray"
@@ -44,7 +44,7 @@
   <xacro:arctos_link
     name="link_4"
-    inertia_origin_xyz="0.0051846 0.10645 0.00064606" inertia_origin_rpy="0 0 0"
-    mass="1.006"
-    ixx="0.062769" ixy="-0.001868" ixz="-3.6977E-05" iyy="0.028683" iyz="0.00032273" izz="0.069443"
+    inertia_origin_xyz="0.0051846 -0.00064606 0.10645" inertia_origin_rpy="0 0 0"
+    mass="14.917"
+    ixx="0.062769" ixy="3.6977E-05" ixz="-0.001868" iyy="0.069443" iyz="-0.00032273" izz="0.028683"
     origin_xyz="0 0 0" origin_rpy="0 0 0"
     material_name="gray"
@@ -52,7 +52,7 @@
   <xacro:arctos_link
     name="link_5"
-    inertia_origin_xyz="-0.00049422 0.0067098 -2.4246E-07" inertia_origin_rpy="0 0 0"
+    inertia_origin_xyz="-0.00049422 2.4246E-07 0.0067098" inertia_origin_rpy="0 0 0"
     mass="0.34309"
-    ixx="0.00034995" ixy="-1.1371E-06" ixz="1.2487E-09" iyy="0.00022745" iyz="1.4302E-09" izz="0.00030039"
+    ixx="0.00034995" ixy="-1.2487E-09" ixz="-1.1371E-06" iyy="0.00030039" iyz="-1.4302E-09" izz="0.00022745"
     origin_xyz="0 0 0" origin_rpy="0 0 0"
     material_name="gray"
@@ -60,7 +60,7 @@
   <xacro:arctos_link
     name="link_6"
-    inertia_origin_xyz="3.1972E-05 0.011587 0" inertia_origin_rpy="0.0 0.0 0.0"
+    inertia_origin_xyz="3.1972E-05 -5.2042E-18 0.011587" inertia_origin_rpy="0.0 0.0 0.0"
     mass="0.068739"
-    ixx="2.0617E-05" ixy="-2.849E-08" ixz="-7.3853E-22" iyy="3.4376E-05" iyz="2.1018E-21" izz="2.0453E-05"
+    ixx="2.0617E-05" ixy="-1.6907E-20" ixz="-2.849E-08" iyy="2.0453E-05" iyz="2.0027E-21" izz="3.4376E-05"
     origin_xyz="0 0 0" origin_rpy="0 0 0"
     material_name="gray"
@@ -86,11 +86,11 @@
     origin_xyz="0 0.029976 0.36377" origin_rpy="0 0 0"
     axis_xyz="-1 0 0"
-    limit_l="-2.0769" limit_u="1.5" limit_e="1" limit_v="3.4907" mimic=""
+    limit_l="-2.0769" limit_u="2.949606436" limit_e="1" limit_v="3.4907" mimic=""
   />
   <xacro:arctos_joint
     name="A_joint" type="revolute"
     parent="link_3" child="link_4"
-    origin_xyz="0.048 0.198 0.09" origin_rpy="0 0 0"
-    axis_xyz="0.0 1.0 0.0"
+    origin_xyz="0.048 -0.09 0.198" origin_rpy="0 0 0"
+    axis_xyz="0 0 1"
     limit_l="-3.3161" limit_u="3.3161" limit_e="1" limit_v="5.236" mimic=""
   />
@@ -98,5 +98,5 @@
     name="B_joint" type="revolute"
     parent="link_4" child="link_5"
-    origin_xyz="0 0.207 0" origin_rpy="0 0 0"
+    origin_xyz="0 0 0.207" origin_rpy="0 0 0"
     axis_xyz="1 0 0"
     limit_l="-2.0944" limit_u="2.0944" limit_e="1" limit_v="5.236" mimic=""
@@ -105,6 +105,6 @@
     name="C_joint" type="revolute"
     parent="link_5" child="link_6"
-    origin_xyz="0 0.052 0" origin_rpy="0 0 0"
-    axis_xyz="0.0 1.0 0.0"
+    origin_xyz="0 0 0.052" origin_rpy="0 0 0"
+    axis_xyz="0.0 0.0 1.0"
     limit_l="-6.2832" limit_u="6.2832" limit_e="1" limit_v="8.3776" mimic=""
   />

File: arctos_moveit_config/config/arctos.ros2_control.xacro (robot description, xacro)
@@ -14,5 +14,5 @@
           <plugin>arctos_interface/ArctosInterface</plugin>
           <param name="device">/dev/ttyUSB0</param>
-          <param name="baud_rate">57600</param>
+          <param name="baud_rate">19200</param>
           <param name="timeout">1000</param>
         </xacro:unless>
