Commit message: use Moveit setup assistant to generate new "moveit_config" with gripper

File: arctos_moveit_config/config/arctos.ros2_control.xacro (robot description, xacro)
@@ -1,5 +1,7 @@
 <?xml version="1.0"?>
 <robot xmlns:xacro="http://www.ros.org/wiki/xacro">
-  <xacro:macro name="arctos_ros2_control" params="name">
+  <xacro:macro name="arctos_ros2_control" params="name initial_positions_file">
+    <xacro:property name="initial_positions"
+      value="${load_yaml(initial_positions_file)['initial_positions']}" />
     <ros2_control name="${name}" type="system">
       <hardware>
@@ -8,13 +10,13 @@
       <joint name="X_joint">
         <command_interface name="position">
-          <param name="min">{-2*pi}</param>
-          <param name="max">{2*pi}</param>
+          <!-- <param name="min">{-2*pi}</param>
+          <param name="max">{2*pi}</param> -->
         </command_interface>
         <command_interface name="velocity">
-          <param name="min">-3.15</param>
-          <param name="max">3.15</param>
+          <!-- <param name="min">-3.15</param>
+          <param name="max">3.15</param> -->
         </command_interface>
         <state_interface name="position">
-          <param name="initial_value">0.0</param>
+          <param name="initial_value">${initial_positions['X_joint']}</param>
         </state_interface>
         <state_interface name="velocity" />
@@ -22,13 +24,13 @@
       <joint name="Y_joint">
         <command_interface name="position">
-          <param name="min">{-2*pi}</param>
-          <param name="max">{2*pi}</param>
+          <!-- <param name="min">{-2*pi}</param>
+          <param name="max">{2*pi}</param> -->
         </command_interface>
         <command_interface name="velocity">
-          <param name="min">-3.15</param>
-          <param name="max">3.15</param>
+          <!-- <param name="min">-3.15</param>
+          <param name="max">3.15</param> -->
         </command_interface>
         <state_interface name="position">
-          <param name="initial_value">0.0</param>
+          <param name="initial_value">${initial_positions['Y_joint']}</param>
         </state_interface>
         <state_interface name="velocity" />
@@ -36,13 +38,13 @@
       <joint name="Z_joint">
         <command_interface name="position">
-          <param name="min">{-pi}</param>
-          <param name="max">{pi}</param>
+          <!-- <param name="min">{-pi}</param>
+          <param name="max">{pi}</param> -->
         </command_interface>
         <command_interface name="velocity">
-          <param name="min">-3.15</param>
-          <param name="max">3.15</param>
+          <!-- <param name="min">-3.15</param>
+          <param name="max">3.15</param> -->
         </command_interface>
         <state_interface name="position">
-          <param name="initial_value">0.0</param>
+          <param name="initial_value">${initial_positions['Z_joint']}</param>
         </state_interface>
         <state_interface name="velocity" />
@@ -50,13 +52,13 @@
       <joint name="A_joint">
         <command_interface name="position">
-          <param name="min">{-2*pi}</param>
-          <param name="max">{2*pi}</param>
+          <!-- <param name="min">{-2*pi}</param>
+          <param name="max">{2*pi}</param> -->
         </command_interface>
         <command_interface name="velocity">
-          <param name="min">-3.2</param>
-          <param name="max">3.2</param>
+          <!-- <param name="min">-3.2</param>
+          <param name="max">3.2</param> -->
         </command_interface>
         <state_interface name="position">
-          <param name="initial_value">0.0</param>
+          <param name="initial_value">${initial_positions['A_joint']}</param>
         </state_interface>
         <state_interface name="velocity" />
@@ -64,13 +66,13 @@
       <joint name="B_joint">
         <command_interface name="position">
-          <param name="min">{-2*pi}</param>
-          <param name="max">{2*pi}</param>
+          <!-- <param name="min">{-2*pi}</param>
+          <param name="max">{2*pi}</param> -->
         </command_interface>
         <command_interface name="velocity">
-          <param name="min">-3.2</param>
-          <param name="max">3.2</param>
+          <!-- <param name="min">-3.2</param>
+          <param name="max">3.2</param> -->
         </command_interface>
         <state_interface name="position">
-          <param name="initial_value">0.0</param>
+          <param name="initial_value">${initial_positions['B_joint']}</param>
         </state_interface>
         <state_interface name="velocity" />
@@ -78,24 +80,32 @@
       <joint name="C_joint">
         <command_interface name="position">
-          <param name="min">{-2*pi}</param>
-          <param name="max">{2*pi}</param>
+          <!-- <param name="min">{-2*pi}</param>
+          <param name="max">{2*pi}</param> -->
         </command_interface>
         <command_interface name="velocity">
-          <param name="min">-3.2</param>
-          <param name="max">3.2</param>
+          <!-- <param name="min">-3.2</param>
+          <param name="max">3.2</param> -->
         </command_interface>
         <state_interface name="position">
-          <param name="initial_value">0.0</param>
+          <param name="initial_value">${initial_positions['C_joint']}</param>
         </state_interface>
         <state_interface name="velocity" />
       </joint>
-      <sensor name="tcp_fts_sensor">
-        <state_interface name="force.x" />
-        <state_interface name="force.y" />
-        <state_interface name="force.z" />
-        <state_interface name="torque.x" />
-        <state_interface name="torque.y" />
-        <state_interface name="torque.z" />
-      </sensor>
+      <joint name="Left_jaw_joint">
+        <command_interface name="position" />
+        <command_interface name="velocity" />
+        <state_interface name="position">
+          <param name="initial_value">${initial_positions['Left_jaw_joint']}</param>
+        </state_interface>
+        <state_interface name="velocity" />
+      </joint>
+      <joint name="Right_jaw_joint">
+        <command_interface name="position" />
+        <command_interface name="velocity" />
+        <state_interface name="position">
+          <param name="initial_value">${initial_positions['Right_jaw_joint']}</param>
+        </state_interface>
+        <state_interface name="velocity" />
+      </joint>
     </ros2_control>
   </xacro:macro>

File: arctos_moveit_config/config/arctos.urdf.xacro (robot description, xacro)
@@ -1,9 +1,9 @@
 <?xml version="1.0"?>
 <robot xmlns:xacro="http://www.ros.org/wiki/xacro" name="arctos">
-    <!-- <xacro:arg name="initial_positions_file" default="initial_positions.yaml" /> -->
+    <xacro:arg name="initial_positions_file" default="initial_positions.yaml" />
     <!-- Import arctos urdf file -->
-    <xacro:include filename="$(find arctos_description)/urdf/arctos.xacro" />
+    <xacro:include filename="$(find arctos_description)/urdf/arctos.urdf" />
     <!-- Import control_xacro -->
-    <!-- <xacro:include filename="arctos.ros2_control.xacro" /> -->
+    <xacro:include filename="arctos.ros2_control.xacro" />
     <!-- <xacro:arctos_ros2_control name="FakeSystem" initial_positions_file="$(arg initial_positions_file)"/> -->
 </robot>
